File: アノレパイソ.kicad_pcb (KiCad board)
At the start: 2 copper layers, 178 x 50 mm, 29 parts, among them SW0 RotaryEncoder_Switch, SW1 SW_PUSH, SW2 SW_PUSH, SW3 SW_PUSH, SW4 SW_PUSH, SW5 SW_PUSH, SW6 SW_PUSH, SW9 SW_PUSH, U1 SO1602AWWB-UC-WB-U, U3 ProMicro

Commit message: 前夜祭更新
Parts:
- moved SW0 7.89 mm to (124.0, 75.0), turned to 0 degrees
- moved U3 4.50 mm to (204.5, 75.0)
- moved U1 0.10 mm to (184.0, 75.0)
- turned SW9 to 0 degrees
Connections:
- SW0 pad S1: (no net) -> Net-(D0-A)
- SW0 pad S2: (no net) -> Col0
Routing:
- net Col0: track 85.2 -> 104.4 mm
- net RE_A: track 63.0 -> 79.8 mm
- net VCC: track 316.3 -> 329.3 mm
- net Col2: track 257.0 -> 267.2 mm
- net GND: track 460.9 -> 451.6 mm
- net SDA: track 38.3 -> 47.3 mm
- net Col3: track 222.5 -> 231.5 mm
- net Reset: track 37.1 -> 46.1 mm
- net Col1: track 317.5 -> 325.9 mm
- net SCL: track 38.3 -> 44.2 mm
- net Row2: track 126.7 -> 131.2 mm
- net Row1: track 130.6 -> 134.9 mm
- net Row0: track 61.7 -> 65.6 mm
- net RE_B: track 65.6 -> 63.0 mm
- net Net-(D0-A): track 6.82 -> 4.53 mm
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Other:
- outline, holes or cut-outs redrawn
- board text removed: "EC12D1524406は、EC12Eのフットプリントとサイズが合わない。"
- board text removed: "EC12E24404A8は、A12Eのフットプリントと異なり、そもそもキースイッチがない。"

Commit message: 基板で暫定表面・裏面を作った。
Parts:
- added SW1: SW_PUSH, kbd-main:keyswitch_cherrymx_hotswap_1u, B.Cu at (56.4, 150.5)
- added SW2: SW_PUSH, kbd-main:keyswitch_cherrymx_hotswap_1u, B.Cu at (75.4, 150.5)
- added SW3: SW_PUSH, kbd-main:keyswitch_cherrymx_hotswap_1u, B.Cu at (94.4, 150.5)
- added SW4: SW_PUSH, kbd-main:keyswitch_cherrymx_hotswap_1u, B.Cu at (56.4, 169.5)
- added SW5: SW_PUSH, kbd-main:keyswitch_cherrymx_hotswap_1u, B.Cu at (75.4, 169.6)
- added SW6: SW_PUSH, kbd-main:keyswitch_cherrymx_hotswap_1u, B.Cu at (94.4, 169.6)
- moved SW4 25.0 mm to (56.4, 59.5)
- moved D0 25.0 mm to (133.3, 57.8)
- moved D1 25.0 mm to (64.5, 47.8)
- moved D2 25.0 mm to (83.5, 47.8)
- moved D3 25.0 mm to (102.5, 47.8)
- moved D4 25.0 mm to (64.5, 52.2)
- moved D5 25.0 mm to (83.5, 52.2)
- moved D6 25.0 mm to (102.5, 52.4)
- moved LED1 25.0 mm to (136.0, 62.0)
- moved LED10 25.0 mm to (106.5, 32.5)
- moved LED11 25.0 mm to (112.0, 38.0)
- moved LED12 25.0 mm to (136.0, 38.0)
- moved LED2 25.0 mm to (112.0, 62.0)
- moved LED3 25.0 mm to (106.5, 67.5)
- moved LED4 25.0 mm to (94.4, 64.3)
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Routing:
- net Net-(D3-A): track 16.0 -> 17.2 mm
Other:
- board size 178 x 50 mm -> 178 x 160 mm

Commit message: 鶴野さん出社最終日前に更新。
Parts:
- SW1, SW2, SW3, SW4, SW5, SW6: footprint kbd-main:keyswitch_cherrymx_hotswap_1u -> kbd_SW_Hole:SW_Hole_1u
- moved SW9 16.3 mm to (167.5, 72.0)
Routing:
- net Reset: track 46.1 -> 62.6 mm
- net Net-(D3-A): track 17.2 -> 16.0 mm
- net GND: track 451.6 -> 452.2 mm
Other:
- outline, holes or cut-outs redrawn
- board text added: "Perfecting Art of Electrowiring"
- board text added: "基板"
- board text added: "底板"
- board text added: "表板"
- board text removed: "Perfecting Art of Electrowireing"
